Commit message: Generated new ANYtree urdf. Also halved z-axis base velocity limit in motion plans

File: anytree_description/urdf/anytree.urdf (robot description, URDF)
Before this commit: robot anymal, 89 links, 88 joints
Links:
- added link camera_accel_frame
- added link camera_accel_optical_frame
- added link camera_bottom_screw_frame
- added link camera_color_frame
- added link camera_color_optical_frame
- added link camera_depth_frame
- added link camera_depth_optical_frame
- added link camera_gyro_frame
- added link camera_gyro_optical_frame
- added link camera_infra1_frame
- added link camera_infra1_optical_frame
- added link camera_infra2_frame
- added link camera_infra2_optical_frame
- added link camera_link, mass 0.072; collision box size=0.02505 0.09 0.025; visual mesh filename=package://realsense2_description/meshes/d435.dae
- added link hatch_top, mass 0.1; collision box size=0.1495 0.108 0.02; visual box size=0.1495 0.108 0.02
- added link unitree_realsense_mount; visual mesh filename=package://anymal_coyote_drs/urdf/modules/unitree_z1/unitree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
- link hatch_unitree_support: mass None -> 0.5; geometry collision box size=0.098 0.19 0.01; visual box size=0.098 0.19 0.01
- link unitree_mount: geometry 
Joints:
- removed joint hatch_to_hatch_unitree_support
- added joint camera_accel_joint: type fixed, parent camera_link, child camera_accel_frame, origin xyz=-0.01174 -0.00552 0.0051 rpy=0 0 0
- added joint camera_accel_optical_joint: type fixed, parent camera_accel_frame, child camera_accel_optical_frame, origin xyz=0 0 0 rpy=-1.5707963267948966 0 -1.5707963267948966
- added joint camera_color_joint: type fixed, parent camera_link, child camera_color_frame, origin xyz=0 0.015 0 rpy=0 0 0
- added joint camera_color_optical_joint: type fixed, parent camera_color_frame, child camera_color_optical_frame, origin xyz=0 0 0 rpy=-1.5707963267948966 0 -1.5707963267948966
- added joint camera_depth_joint: type fixed, parent camera_link, child camera_depth_frame, origin xyz=0 0 0 rpy=0 0 0
- added joint camera_depth_optical_joint: type fixed, parent camera_depth_frame, child camera_depth_optical_frame, origin xyz=0 0 0 rpy=-1.5707963267948966 0 -1.5707963267948966
- added joint camera_gyro_joint: type fixed, parent camera_link, child camera_gyro_frame, origin xyz=-0.01174 -0.00552 0.0051 rpy=0 0 0
- added joint camera_gyro_optical_joint: type fixed, parent camera_gyro_frame, child camera_gyro_optical_frame, origin xyz=0 0 0 rpy=-1.5707963267948966 0 -1.5707963267948966
- added joint camera_infra1_joint: type fixed, parent camera_link, child camera_infra1_frame, origin xyz=0 0.0 0 rpy=0 0 0
- added joint camera_infra1_optical_joint: type fixed, parent camera_infra1_frame, child camera_infra1_optical_frame, origin xyz=0 0 0 rpy=-1.5707963267948966 0 -1.5707963267948966
- added joint camera_infra2_joint: type fixed, parent camera_link, child camera_infra2_frame, origin xyz=0 -0.05 0 rpy=0 0 0
- added joint camera_infra2_optical_joint: type fixed, parent camera_infra2_frame, child camera_infra2_optical_frame, origin xyz=0 0 0 rpy=-1.5707963267948966 0 -1.5707963267948966
- added joint camera_joint: type fixed, parent unitree_realsense_mount, child camera_bottom_screw_frame, origin xyz=0.008 0.0 0.0375 rpy=0.0 0.0 0.0
- added joint camera_link_joint: type fixed, parent camera_bottom_screw_frame, child camera_link, origin xyz=0.010600000000000002 0.0175 0.0125 rpy=0 0 0
- added joint hand_to_unitree_realsense_mount_joint: type fixed, parent link06, child unitree_realsense_mount, origin xyz=0.0365 0.0 0.0 rpy=0.0 0.0 0.0
- added joint hatch_to_hatch_top: type fixed, parent hatch, child hatch_top, origin xyz=0.0 0.0 0.015 rpy=0.0 0.0 0.0
- added joint hatch_top_to_hatch_unitree_support: type fixed, parent hatch_top, child hatch_unitree_support, origin xyz=0.02525 0.0 0.015 rpy=0.0 0.0 0.0
- joint hatch_unitree_support_to_unitree_mount: origin xyz=0.0 0.0 0.0 rpy=0 0 0 -> xyz=0 0 0.005 rpy=0 0 0
